Commit message: cmd_vel and joint publishing work

File: car_description/robot/red_crash.urdf.xacro (robot description, xacro)
@@ -1,13 +1,18 @@
 <?xml version="1.0"?>
 <robot xmlns:xacro="http://ros.org/wiki/xacro" name="car">
-  <xacro:arg name="wheel_diameter" default="0.112"/>
+  <xacro:arg name="wheel_diameter" default="0.120"/>
+  <xacro:property name="update_rate" default="20"/>
   <xacro:property name="wheel_radius" value="${$(arg wheel_diameter)/2}"/>
-  <xacro:property name="wheel_width" value="0.047"/>
+  <xacro:property name="wheel_width" value="0.032"/>
+  <xacro:property name="wheel_mass" value="0.1"/>
+  <xacro:property name="omni_wheel_radius" value="${wheel_radius}"/>
+  <xacro:property name="omni_wheel_width" value="0.029"/>
+  <xacro:property name="omni_wheel_mass" value="${wheel_mass}"/>
+  <xacro:property name="omni_vertical_offset" value="0.005"/>
   <xacro:property name="wheel_friction" value="0.8"/>
   <xacro:property name="wheelbase_length" value="0.3429"/>
   <xacro:property name="front_wheelbase_width" value="0.25"/>
   <xacro:property name="rear_wheelbase_width" value="0.25"/>
-  <xacro:property name="wheel_mass" value="0.1"/>
-  <xacro:property name="total_mass" value = "3.0"/>
+  <xacro:property name="total_mass" value = "5.0"/>
   <xacro:property name="shock_travel" value = "0.09"/>
   <!-- see https://www.gobilda.com/beeline-chassis-kit/ -->
@@ -17,4 +22,9 @@
   <xacro:property name="chassis_elevation" value = "-0.01"/>
   <xacro:property name="chassis_mass" value = "${total_mass-4*wheel_mass}"/>
+  <!-- all the batteries, pi, etc. are represented by one box -->>
+  <xacro:property name="components_height" value = "0.04"/>
+  <xacro:property name="components_width" value = "0.30"/>
+  <xacro:property name="components_length" value = "0.15"/>
+  <xacro:property name="components_mass" value = "2.0"/>
   <!-- wheelbase is to wheel centers -->
   <xacro:property name="wheelbase_width" value = "${chassis_width+wheel_width}"/>
@@ -58,30 +68,55 @@
         <cylinder_inertial m="${wheel_mass}" r="${wheel_radius}" h="${wheel_width}"/>
     </link>
-  </xacro:macro>
-  <link name="dummy">
+    <gazebo reference="${name}">
+        <mu1>${wheel_friction}</mu1>
+        <material>Gazebo/DarkGrey</material>
+    </gazebo>
+  </xacro:macro>
+  <xacro:macro name="xbox" params="name length width height mass">
+    <link name="${name}">
+        <visual>
+        <geometry>
+            <box size="${length} ${width} ${height}"/>
+        </geometry>
+        </visual>
+        <collision>
+        <geometry>
+            <box size="${length} ${width} ${height}"/>
+        </geometry>
+        </collision>
+        <inertial>
+        <mass value="${mass}"/>
+        <box_inertia m="${mass}" x="${length}" y="${width}" z="${height}"/>
+        </inertial>
+    </link>
+  </xacro:macro>
+  <xacro:macro name="omni_wheel" params="name" >
+    <link name="${name}">
+        <visual>
+        <geometry>
+            <cylinder length="${omni_wheel_width}" radius="${omni_wheel_radius}"/>
+        </geometry>
+        <material name="black">
+            <color rgba="0 0 0 1"/>
+        </material>
+        </visual>
+        <collision>
+        <geometry>
+            <cylinder length="${omni_wheel_width}" radius="${omni_wheel_radius}"/>
+        </geometry>
+        </collision>
+        <cylinder_inertial m="${wheel_mass}" r="${omni_wheel_radius}" h="${omni_wheel_width}"/>
+    </link>
+    <gazebo reference="${name}">
+        <mu1>${wheel_friction}</mu1>
+        <mu2>0.0}</mu2>
+        <material>Gazebo/Grey</material>
+    </gazebo>
+  </xacro:macro>
+  <link name="base_footprint">
    </link>
   <link name="base_link">
-    <visual>
-      <origin xyz="0 0 0.1" rpy="0 0 0"/>
-      <geometry>
-        <cylinder length="0.2" radius="0.01"/>
-      </geometry>
-      <material name="silver">
-        <color rgba="0.75 0.75 0.75 1"/>
-      </material>
-    </visual>
-    <collision>
-      <origin xyz="0 0 0.1" rpy="0 0 0"/>
-      <geometry>
-        <cylinder length="0.2" radius="0.01"/>
-      </geometry>
-    </collision>
-    <inertial>
-      <mass value="0.01"/>
-      <inertia ixx="0.015" iyy="0.0375" izz="0.0375"
-               ixy="0" ixz="0" iyz="0"/>
-    </inertial>
   </link>
-  <link name="chassis_link">
+  <link name="chassis">
     <visual>
       <geometry>
@@ -99,6 +134,8 @@
     </inertial>
   </link>
-  <wheel name="back_left_wheel"></wheel>
-  <wheel name="back_right_wheel"></wheel>
+  <xbox name="components" length="${components_length}" width="${components_width}" height="${components_height}" mass="${components_mass}">
+  </xbox>
+  <omni_wheel name="back_left_wheel"></omni_wheel>
+  <omni_wheel name="back_right_wheel"></omni_wheel>
   <wheel name="mid_left_wheel"></wheel>
   <wheel name="mid_right_wheel"></wheel>
@@ -158,6 +195,6 @@
     </sensor>
   </gazebo>
-  <joint name="dummy_joint" type="fixed">
-     <parent link="dummy"/>
+  <joint name="base_link_joint" type="fixed">
+     <parent link="base_footprint"/>
      <child link="base_link"/>
     <origin rpy="0 0 0" xyz="0 0 ${wheel_radius/2}"/>
@@ -165,19 +202,19 @@
   <joint name="back_left_wheel_joint" type="continuous">
     <axis xyz="0 0 1"/>
-    <parent link="chassis_link"/>
+    <parent link="chassis"/>
     <child link="back_left_wheel"/>
-    <origin rpy="${-pi/2} 0 0" xyz="${-wheelbase_length/2} ${wheelbase_width/2} 0"/>
+    <origin rpy="${-pi/2} 0 0" xyz="${-wheelbase_length/2} ${wheelbase_width/2} ${omni_vertical_offset}"/>
     <limit effort="10000" velocity="500" />
   </joint>
   <joint name="back_right_wheel_joint" type="continuous">
     <axis xyz="0 0 1"/>
-    <parent link="chassis_link"/>
+    <parent link="chassis"/>
     <child link="back_right_wheel"/>
-    <origin rpy="${-pi/2} 0 0" xyz="${-wheelbase_length/2} -${wheelbase_width/2} 0"/>
+    <origin rpy="${-pi/2} 0 0" xyz="${-wheelbase_length/2} -${wheelbase_width/2} ${omni_vertical_offset}"/>
     <limit effort="10000" velocity="500" />
   </joint>
   <joint name="mid_left_wheel_joint" type="continuous">
     <axis xyz="0 0 1"/>
-    <parent link="chassis_link"/>
+    <parent link="chassis"/>
     <child link="mid_left_wheel"/>
     <origin rpy="${-pi/2} 0 0" xyz="0 ${wheelbase_width/2} 0"/>
@@ -186,5 +223,5 @@
   <joint name="mid_right_wheel_joint" type="continuous">
     <axis xyz="0 0 1"/>
-    <parent link="chassis_link"/>
+    <parent link="chassis"/>
     <child link="mid_right_wheel"/>
     <origin rpy="${-pi/2} 0 0" xyz="0 ${-wheelbase_width/2} 0"/>
@@ -193,5 +230,5 @@
   <joint name="front_left_wheel_joint" type="continuous">
     <axis xyz="0 0 1"/>
-    <parent link="chassis_link"/>
+    <parent link="chassis"/>
     <child link="front_left_wheel"/>
     <origin rpy="${-pi/2} 0 0" xyz="${wheelbase_length/2} ${wheelbase_width/2} 0"/>
@@ -200,5 +237,5 @@
   <joint name="front_right_wheel_joint" type="continuous">
     <axis xyz="0 0 1"/>
-    <parent link="chassis_link"/>
+    <parent link="chassis"/>
     <child link="front_right_wheel"/>
     <origin rpy="${-pi/2} 0 0" xyz="${wheelbase_length/2} ${-wheelbase_width/2} 0"/>
@@ -207,7 +244,60 @@
   <joint name="chassis_joint" type="fixed">
     <parent link="base_link"/>
-    <child link="chassis_link"/>
+    <child link="chassis"/>
     <origin rpy="0 0 0" xyz="0 0 ${wheel_radius/2}"/>
   </joint>
+  <joint name="components_joint" type="fixed">
+    <parent link="chassis"/>
+    <child link="components"/>
+    <origin rpy="0 0 0" xyz="${-wheelbase_length/4} 0 ${(components_height+chassis_height)/2}"/>
+  </joint>
+  <gazebo>
+    <!--
+      couldn't find documentation, found names in https://github.com/ros-simulation/gazebo_ros_pkgs/blob/galactic/gazebo_plugins/src/gazebo_ros_diff_drive.cpp
+      good example here:
+      https://github.com/ros-simulation/gazebo_ros_pkgs/blob/galactic/gazebo_plugins/test/worlds/gazebo_ros_diff_drive.world
+    -->
+    <plugin name="differential_drive_controller" filename="libgazebo_ros_diff_drive.so">
+        <ros>
+          <!-- <namespace></namespace> -->
+          <remapping>cmd_vel:=cmd_vel</remapping>
+          <remapping>odom:=odom</remapping>
+        </ros>
+      <!-- Plugin update rate in Hz -->
+      <update_rate>${update_rate}</update_rate>
+      <!-- Name of left joint, defaults to `left_joint` -->
+      <left_joint>mid_left_wheel_joint</left_joint>
+      <leftJoint>mid_left_wheel_joint</leftJoint>
+      <!-- Name of right joint, defaults to `right_joint` -->
+      <right_joint>mid_right_wheel_joint</right_joint>
+      <rightJoint>mid_right_wheel_joint</rightJoint>
+      <!-- The distance from the center of one wheel to the other, in meters, defaults to 0.34 m -->
+      <wheel_separation>${wheelbase_width}</wheel_separation>
+      <!-- Diameter of the wheels, in meters, defaults to 0.15 m -->
+      <wheel_diameter>${wheel_radius * 2.0}</wheel_diameter>
+      <!-- Wheel acceleration, in rad/s^2, defaults to 0.0 rad/s^2 -->
+      <max_wheel_acceleration>5.0</max_wheel_acceleration>
+      <!-- Maximum torque which the wheels can produce, in Nm, defaults to 5 Nm -->
+      <max_wheel_torque>2.4</max_wheel_torque>
+      <!-- Topic to receive geometry_msgs/Twist message commands, defaults to `cmd_vel` -->
+      <commandTopic>cmd_vel</commandTopic>
+      <!-- Topic to publish nav_msgs/Odometry messages, defaults to `odom` -->
+      <odometryTopic>odom</odometryTopic>
+      <!-- Odometry frame, defaults to `odom` -->
+      <odometry_frame>odom</odometry_frame>
+      <!-- Robot frame to calculate odometry from, defaults to `base_footprint` -->
+      <robot_base_frame>base_footprint</robot_base_frame>
+      <!-- Odometry source, 0 for ENCODER, 1 for WORLD, defaults to WORLD -->
+      <odometry_source>1</odometry_source>
+      <!-- Set to true to publish transforms for the wheel links, defaults to false -->
+      <publish_wheel_tf>true</publish_wheel_tf>
+      <!-- Set to true to publish transforms for the odometry, defaults to true -->
+      <publish_odom_tf>true</publish_odom_tf>
+      <!-- Set to true to publish sensor_msgs/JointState on /joint_states for the wheel joints, defaults to false -->
+      <publishWheelJointState>true</publishWheelJointState>
+      <!-- Set to true to swap right and left wheels, defaults to true -->
+      <legacyMode>false</legacyMode>
+    </plugin>
+  </gazebo>
   <gazebo>
     <plugin name="gazebo_ros_control" filename="libgazebo_ros_control.so">
@@ -215,21 +305,5 @@
     </plugin>
   </gazebo>
-  <gazebo reference="front_left_wheel">
-    <mu1>${wheel_friction}</mu1>
-    <material>Gazebo/DarkGrey</material>
-  </gazebo>
-  <gazebo reference="front_right_wheel">
-    <mu1>${wheel_friction}</mu1>
-    <material>Gazebo/DarkGrey</material>
-  </gazebo>
-  <gazebo reference="back_left_wheel">
-    <mu1>${wheel_friction}</mu1>
-    <material>Gazebo/DarkGrey</material>
-  </gazebo>
-  <gazebo reference="back_right_wheel">
-    <mu1>${wheel_friction}</mu1>
-    <material>Gazebo/DarkGrey</material>
-  </gazebo>
-  <gazebo reference="chassis_link">
+  <gazebo reference="chassis">
     <material>Gazebo/Red</material>
   </gazebo>

Commit message: red-crash improvements, all wheels drive, etc.

File: car_description/robot/red_crash.urdf.xacro (robot description, xacro)
@@ -14,12 +14,4 @@
   <xacro:property name="front_wheelbase_width" value="0.25"/>
   <xacro:property name="rear_wheelbase_width" value="0.25"/>
-  <xacro:property name="total_mass" value = "5.0"/>
-  <xacro:property name="shock_travel" value = "0.09"/>
-  <!-- see https://www.gobilda.com/beeline-chassis-kit/ -->
-  <xacro:property name="chassis_height" value = "0.048"/>
-  <xacro:property name="chassis_width" value = "0.360"/>
-  <xacro:property name="chassis_length" value = "0.432"/>
-  <xacro:property name="chassis_elevation" value = "-0.01"/>
-  <xacro:property name="chassis_mass" value = "${total_mass-4*wheel_mass}"/>
   <!-- all the batteries, pi, etc. are represented by one box -->>
   <xacro:property name="components_height" value = "0.04"/>
@@ -27,4 +19,9 @@
   <xacro:property name="components_length" value = "0.15"/>
   <xacro:property name="components_mass" value = "2.0"/>
+  <!-- see https://www.gobilda.com/beeline-chassis-kit/ -->
+  <xacro:property name="chassis_height" value = "0.048"/>
+  <xacro:property name="chassis_width" value = "0.360"/>
+  <xacro:property name="chassis_length" value = "0.432"/>
+  <xacro:property name="chassis_mass" value = "4.0"/>
   <!-- wheelbase is to wheel centers -->
   <xacro:property name="wheelbase_width" value = "${chassis_width+wheel_width}"/>
@@ -71,4 +68,25 @@
         <mu1>${wheel_friction}</mu1>
         <material>Gazebo/DarkGrey</material>
+    </gazebo>
+  </xacro:macro>
+  <xacro:macro name="xcylinder" params="name radius length color:='Gazebo/DarkGrey' mass:=0.1" >
+    <link name="${name}">
+        <visual>
+        <geometry>
+            <cylinder length="${length}" radius="${radius}"/>
+        </geometry>
+        <material name="${name}_material">
+            <color rgba="0 0 0 1"/>
+        </material>
+        </visual>
+        <collision>
+        <geometry>
+            <cylinder length="${length}" radius="${radius}"/>
+        </geometry>
+        </collision>
+        <cylinder_inertial m="${mass}" r="${radius}" h="${length}"/>
+    </link>
+    <gazebo reference="${name}">
+        <material>${color}</material>
     </gazebo>
   </xacro:macro>
@@ -142,23 +160,5 @@
   <wheel name="front_left_wheel"></wheel>
   <wheel name="front_right_wheel"></wheel>
-  <link name="laser_scanner_link">
-    <collision>
-      <origin xyz="0 0 0" rpy="0 0 0"/>
-      <geometry>
-        <box size=".127 0.1016 0.0508"/>
-      </geometry>
-    </collision>
-    <visual>
-      <origin xyz="0 0 0" rpy="0 0 0"/>
-      <geometry>
-        <box size=".127 0.1016 0.0508"/>
-      </geometry>
-    </visual>
-    <inertial>
-      <mass value="1e-5"/>
-      <origin xyz="0 0 0" rpy="0 0 0"/>
-      <inertia ixx="1e-6" ixy="0" ixz="0" iyy="1e-6" iyz="0" izz="1e-6"/>
-    </inertial>
-  </link>
+  <xcylinder name="laser_scanner_link" length="0.045" radius="0.040"/>
   <joint name="laser_scanner_joint" type="fixed">
     <origin rpy="0 0 0" xyz="0.1397 0 0.2159"/>
@@ -169,5 +169,5 @@
     <sensor type="ray" name="laser_scanner">
     <always_on>true</always_on>
-    <visualize>true</visualize>
+    <visualize>false</visualize>
     <update_rate>20</update_rate>
     <ray>
@@ -183,5 +183,5 @@
         <min>0.10</min>
         <max>15.0</max>
-        <resolution>0.1</resolution>
+        <resolution>0.01</resolution>
       </range>
     </ray>
@@ -204,5 +204,5 @@
     <parent link="chassis"/>
     <child link="back_left_wheel"/>
-    <origin rpy="${-pi/2} 0 0" xyz="${-wheelbase_length/2} ${wheelbase_width/2} ${omni_vertical_offset}"/>
+    <origin rpy="${-pi/2} 0 0" xyz="${-wheelbase_length/2} ${wheelbase_width/2} 0.0"/>
     <limit effort="10000" velocity="500" />
   </joint>
@@ -211,5 +211,5 @@
     <parent link="chassis"/>
     <child link="back_right_wheel"/>
-    <origin rpy="${-pi/2} 0 0" xyz="${-wheelbase_length/2} -${wheelbase_width/2} ${omni_vertical_offset}"/>
+    <origin rpy="${-pi/2} 0 0" xyz="${-wheelbase_length/2} -${wheelbase_width/2} 0.0"/>
     <limit effort="10000" velocity="500" />
   </joint>
@@ -232,5 +232,5 @@
     <parent link="chassis"/>
     <child link="front_left_wheel"/>
-    <origin rpy="${-pi/2} 0 0" xyz="${wheelbase_length/2} ${wheelbase_width/2} 0"/>
+    <origin rpy="${-pi/2} 0 0" xyz="${wheelbase_length/2} ${wheelbase_width/2} ${omni_vertical_offset}"/>
     <limit effort="10000" velocity="500" />
   </joint>
@@ -239,5 +239,5 @@
     <parent link="chassis"/>
     <child link="front_right_wheel"/>
-    <origin rpy="${-pi/2} 0 0" xyz="${wheelbase_length/2} ${-wheelbase_width/2} 0"/>
+    <origin rpy="${-pi/2} 0 0" xyz="${wheelbase_length/2} ${-wheelbase_width/2} ${omni_vertical_offset}"/>
     <limit effort="10000" velocity="500" />
   </joint>
@@ -262,14 +262,17 @@
           <!-- <namespace></namespace> -->
           <remapping>cmd_vel:=cmd_vel</remapping>
-          <remapping>odom:=odom</remapping>
+          <remapping>odom:=ground_truth/odom</remapping>
         </ros>
       <!-- Plugin update rate in Hz -->
       <update_rate>${update_rate}</update_rate>
+      <num_wheel_pairs>3</num_wheel_pairs>
       <!-- Name of left joint, defaults to `left_joint` -->
       <left_joint>mid_left_wheel_joint</left_joint>
-      <leftJoint>mid_left_wheel_joint</leftJoint>
+      <left_joint>back_left_wheel_joint</left_joint>
+      <left_joint>front_left_wheel_joint</left_joint>
       <!-- Name of right joint, defaults to `right_joint` -->
       <right_joint>mid_right_wheel_joint</right_joint>
-      <rightJoint>mid_right_wheel_joint</rightJoint>
+      <right_joint>back_right_wheel_joint</right_joint>
+      <right_joint>front_right_wheel_joint</right_joint>
       <!-- The distance from the center of one wheel to the other, in meters, defaults to 0.34 m -->
       <wheel_separation>${wheelbase_width}</wheel_separation>
@@ -292,4 +295,5 @@
       <!-- Set to true to publish transforms for the wheel links, defaults to false -->
       <publish_wheel_tf>true</publish_wheel_tf>
+      <publish_odom>true</publish_odom>
       <!-- Set to true to publish transforms for the odometry, defaults to true -->
       <publish_odom_tf>true</publish_odom_tf>
@@ -300,9 +304,10 @@
     </plugin>
   </gazebo>
+<!--
   <gazebo>
     <plugin name="gazebo_ros_control" filename="libgazebo_ros_control.so">
       <robotNamespace>/sim_car</robotNamespace>
     </plugin>
-  </gazebo>
+  </gazebo> -->
   <gazebo reference="chassis">
     <material>Gazebo/Red</material>

Commit message: refactor

File: car_description/robot/red_crash.urdf.xacro (robot description, xacro)
@@ -132,26 +132,8 @@
     </gazebo>
   </xacro:macro>
-  <link name="base_footprint">
-   </link>
-  <link name="base_link">
-  </link>
-  <link name="chassis">
-    <visual>
-      <geometry>
-        <box size="${chassis_length} ${chassis_width} ${chassis_height}"/>
-      </geometry>
-    </visual>
-    <collision>
-      <geometry>
-        <box size="${chassis_length} ${chassis_width} ${chassis_height}"/>
-      </geometry>
-    </collision>
-    <inertial>
-      <mass value="${chassis_mass}"/>
-      <box_inertia m="${chassis_mass}" x="${chassis_length}" y="${chassis_width}" z="${chassis_height}"/>
-    </inertial>
-  </link>
-  <xbox name="components" length="${components_length}" width="${components_width}" height="${components_height}" mass="${components_mass}">
-  </xbox>
+  <link name="base_footprint"/>
+  <link name="base_link"/>
+  <xbox name="chassis" length="${chassis_length}" width="${chassis_width}" height="${chassis_height}" mass="${chassis_mass}"/>
+  <xbox name="components" length="${components_length}" width="${components_width}" height="${components_height}" mass="${components_mass}"/>
   <omni_wheel name="back_left_wheel"></omni_wheel>
   <omni_wheel name="back_right_wheel"></omni_wheel>
@@ -160,11 +142,11 @@
   <wheel name="front_left_wheel"></wheel>
   <wheel name="front_right_wheel"></wheel>
-  <xcylinder name="laser_scanner_link" length="0.045" radius="0.040"/>
+  <xcylinder name="lidar" length="0.045" radius="0.040"/>
   <joint name="laser_scanner_joint" type="fixed">
     <origin rpy="0 0 0" xyz="0.1397 0 0.2159"/>
     <parent link="base_link"/>
-    <child link="laser_scanner_link"/>
-  </joint>
-  <gazebo reference="laser_scanner_link">
+    <child link="lidar"/>
+  </joint>
+  <gazebo reference="lidar">
     <sensor type="ray" name="laser_scanner">
     <always_on>true</always_on>
@@ -181,5 +163,5 @@
       </scan>
       <range>
-        <min>0.10</min>
+        <min>0.20</min>
         <max>15.0</max>
         <resolution>0.01</resolution>
@@ -191,5 +173,5 @@
         </ros>
         <output_type>sensor_msgs/LaserScan</output_type>
-        <frame_name>laser_scanner_link</frame_name>
+        <frame_name>lidar</frame_name>
       </plugin>
     </sensor>
@@ -304,10 +286,4 @@
     </plugin>
   </gazebo>
-<!--
-  <gazebo>
-    <plugin name="gazebo_ros_control" filename="libgazebo_ros_control.so">
-      <robotNamespace>/sim_car</robotNamespace>
-    </plugin>
-  </gazebo> -->
   <gazebo reference="chassis">
     <material>Gazebo/Red</material>
