Commit message: Bringup includes rviz with robot_description

File: car_description/robot/red_crash.urdf.xacro (robot description, xacro)
@@ -70,5 +70,5 @@
     </gazebo>
   </xacro:macro>
-  <xacro:macro name="xcylinder" params="name radius length color:='Gazebo/DarkGrey' mass:=0.1" >
+  <xacro:macro name="xcylinder" params="name radius length color:='Gazebo/DarkGrey' rgba:='0.5 0.5 0.5 1.0' mass:=0.1" >
     <link name="${name}">
         <visual>
@@ -77,5 +77,5 @@
         </geometry>
         <material name="${name}_material">
-            <color rgba="0 0 0 1"/>
+            <color rgba="${rgba}"/>
         </material>
         </visual>
@@ -91,5 +91,5 @@
     </gazebo>
   </xacro:macro>
-  <xacro:macro name="xbox" params="name length width height mass">
+  <xacro:macro name="xbox" params="name length width height mass color:='Gazebo/Gray' rgba:='0.5 0.5 0.5 1.0'">
     <link name="${name}">
         <visual>
@@ -97,4 +97,7 @@
             <box size="${length} ${width} ${height}"/>
         </geometry>
+        <material name="${name}_material">
+            <color rgba="${rgba}"/>
+        </material>
         </visual>
         <collision>
@@ -108,4 +111,7 @@
         </inertial>
     </link>
+    <gazebo reference="${name}">
+      <material>${color}</material>
+    </gazebo>
   </xacro:macro>
   <xacro:macro name="omni_wheel" params="name" >
@@ -115,6 +121,6 @@
             <cylinder length="${omni_wheel_width}" radius="${omni_wheel_radius}"/>
         </geometry>
-        <material name="black">
-            <color rgba="0 0 0 1"/>
+        <material name="gray">
+            <color rgba="0.5 0.5 0.5 1"/>
         </material>
         </visual>
@@ -134,6 +140,6 @@
   <link name="base_footprint"/>
   <link name="base_link"/>
-  <xbox name="chassis" length="${chassis_length}" width="${chassis_width}" height="${chassis_height}" mass="${chassis_mass}"/>
-  <xbox name="components" length="${components_length}" width="${components_width}" height="${components_height}" mass="${components_mass}"/>
+  <xbox name="chassis" length="${chassis_length}" width="${chassis_width}" height="${chassis_height}" mass="${chassis_mass}" color="Gazebo/Red" rgba="1 0 0 1" />
+  <xbox name="components" length="${components_length}" width="${components_width}" height="${components_height}" mass="${components_mass}" color="Gazebo/Gray"  rgba="0.5 0.5 0.5 1" />
   <omni_wheel name="back_left_wheel"></omni_wheel>
   <omni_wheel name="back_right_wheel"></omni_wheel>
@@ -230,7 +236,7 @@
   </joint>
   <joint name="components_joint" type="fixed">
-    <parent link="chassis"/>
+    <parent link="base_link"/>
     <child link="components"/>
-    <origin rpy="0 0 0" xyz="${-wheelbase_length/4} 0 ${(components_height+chassis_height)/2}"/>
+    <origin rpy="0 0 0" xyz="${-wheelbase_length/4} 0 ${(components_height+chassis_height+wheel_radius)/2}"/>
   </joint>
   <gazebo>
@@ -286,7 +292,4 @@
     </plugin>
   </gazebo>
-  <gazebo reference="chassis">
-    <material>Gazebo/Red</material>
-  </gazebo>
   <gazebo reference="base_link">
     <dampingFactor>0.00007</dampingFactor>
