Commit message: Ackermann simulation connected and runs.

File: car_description/robot/car.urdf.xacro (robot description, xacro)
@@ -32,9 +32,10 @@
     <inertial>
       <mass value="${m}"/>
-      <cylinder_inertia m="${m}" r="${r}" h="${h}"/>
+      <xacro:cylinder_inertia m="${m}" r="${r}" h="${h}"/>
     </inertial>
   </xacro:macro>
-  <link name="dummy">
-   </link>
+  <link name="base_footprint"/>
+  <link name="base_link"/>
+<!--
   <link name="base_link">
     <visual>
@@ -59,4 +60,5 @@
     </inertial>
   </link>
+-->
   <link name="chassis_link">
     <visual>
@@ -72,5 +74,5 @@
     <inertial>
       <mass value="${chassis_mass}"/>
-      <box_inertia m="${chassis_mass}" x="${wheelbase_length}" y="${front_wheelbase_width}" z="${chassis_height}"/>
+      <xacro:box_inertia m="${chassis_mass}" x="${wheelbase_length}" y="${front_wheelbase_width}" z="${chassis_height}"/>
     </inertial>
   </link>
@@ -89,5 +91,5 @@
       </geometry>
     </collision>
-    <cylinder_inertial m="${wheel_mass}" r="${wheel_radius}" h="${wheel_width}"/>
+    <xacro:cylinder_inertial m="${wheel_mass}" r="${wheel_radius}" h="${wheel_width}"/>
   </link>
   <link name="laser_scanner_link">
@@ -110,14 +112,9 @@
     </inertial>
   </link>
-  <joint name="laser_scanner_joint" type="fixed">
-    <origin rpy="0 0 0" xyz="0.1397 0 0.2159"/>
-    <parent link="base_link"/>
-    <child link="laser_scanner_link"/>
-  </joint>
   <gazebo reference="laser_scanner_link">
     <sensor type="ray" name="laser_scanner">
     <always_on>true</always_on>
     <visualize>true</visualize>
-    <update_rate>20</update_rate>
+    <update_rate>8</update_rate>
     <ray>
       <scan>
@@ -158,5 +155,5 @@
       </geometry>
     </collision>
-    <cylinder_inertial m="${wheel_mass}" r="${wheel_radius}" h="${wheel_width}"/>
+    <xacro:cylinder_inertial m="${wheel_mass}" r="${wheel_radius}" h="${wheel_width}"/>
   </link>
   <link name="front_left_wheel_steer">
@@ -194,5 +191,5 @@
       </geometry>
     </collision>
-    <cylinder_inertial m="${wheel_mass}" r="${wheel_radius}" h="${wheel_width}"/>
+    <xacro:cylinder_inertial m="${wheel_mass}" r="${wheel_radius}" h="${wheel_width}"/>
   </link>
   <link name="front_right_wheel_steer">
@@ -230,5 +227,5 @@
       </geometry>
     </collision>
-    <cylinder_inertial m="${wheel_mass}" r="${wheel_radius}" h="${wheel_width}"/>
+    <xacro:cylinder_inertial m="${wheel_mass}" r="${wheel_radius}" h="${wheel_width}"/>
   </link>
   <link name="back_left_wheel_shock">
@@ -254,8 +251,80 @@
     </inertial>
   </link>
-  <joint name="dummy_joint" type="fixed">
-     <parent link="dummy"/>
+  <link name="back_right_wheel_shock">
+    <visual>
+    <origin xyz="0 0 0.1" rpy="0 0 0"/>
+    <geometry>
+      <cylinder length="0.2" radius="0.01"/>
+    </geometry>
+    <material name="silver">
+      <color rgba="0.75 0.75 0.75 1"/>
+    </material>
+  </visual>
+  <collision>
+    <origin xyz="0 0 0.1" rpy="0 0 0"/>
+    <geometry>
+      <cylinder length="0.2" radius="0.01"/>
+    </geometry>
+  </collision>
+  <inertial>
+    <mass value="0.01"/>
+    <inertia ixx="0.015" iyy="0.0375" izz="0.0375"
+              ixy="0" ixz="0" iyz="0"/>
+  </inertial>
+</link>
+  <link name="front_left_wheel_shock">
+      <visual>
+      <origin xyz="0 0 0.1" rpy="0 0 0"/>
+      <geometry>
+        <cylinder length="0.2" radius="0.01"/>
+      </geometry>
+      <material name="silver">
+        <color rgba="0.75 0.75 0.75 1"/>
+      </material>
+    </visual>
+    <collision>
+      <origin xyz="0 0 0.1" rpy="0 0 0"/>
+      <geometry>
+        <cylinder length="0.2" radius="0.01"/>
+      </geometry>
+    </collision>
+    <inertial>
+      <mass value="0.01"/>
+      <inertia ixx="0.015" iyy="0.0375" izz="0.0375"
+               ixy="0" ixz="0" iyz="0"/>
+    </inertial>
+  </link>
+  <link name="front_right_wheel_shock">
+      <visual>
+      <origin xyz="0 0 0.1" rpy="0 0 0"/>
+      <geometry>
+        <cylinder length="0.2" radius="0.01"/>
+      </geometry>
+      <material name="silver">
+        <color rgba="0.75 0.75 0.75 1"/>
+      </material>
+    </visual>
+    <collision>
+      <origin xyz="0 0 0.1" rpy="0 0 0"/>
+      <geometry>
+        <cylinder length="0.2" radius="0.01"/>
+      </geometry>
+    </collision>
+    <inertial>
+      <mass value="0.01"/>
+      <inertia ixx="0.015" iyy="0.0375" izz="0.0375"
+               ixy="0" ixz="0" iyz="0"/>
+    </inertial>
+  </link>
+  <joint name="base_link_joint" type="fixed">
+     <parent link="base_footprint"/>
      <child link="base_link"/>
+     <origin rpy="0 0 0" xyz="0 0 0"/>
    </joint>
+   <joint name="laser_scanner_joint" type="fixed">
+    <origin rpy="0 0 0" xyz="0.1397 0 0.2159"/>
+    <parent link="base_link"/>
+    <child link="laser_scanner_link"/>
+  </joint>
   <joint name="back_left_shock_joint" type="prismatic">
     <limit lower="0" upper="${shock_travel}" effort="100" velocity="100"/>
@@ -272,26 +341,4 @@
     <limit effort="10000" velocity="500" />
   </joint>
-  <link name="back_right_wheel_shock">
-      <visual>
-      <origin xyz="0 0 0.1" rpy="0 0 0"/>
-      <geometry>
-        <cylinder length="0.2" radius="0.01"/>
-      </geometry>
-      <material name="silver">
-        <color rgba="0.75 0.75 0.75 1"/>
-      </material>
-    </visual>
-    <collision>
-      <origin xyz="0 0 0.1" rpy="0 0 0"/>
-      <geometry>
-        <cylinder length="0.2" radius="0.01"/>
-      </geometry>
-    </collision>
-    <inertial>
-      <mass value="0.01"/>
-      <inertia ixx="0.015" iyy="0.0375" izz="0.0375"
-               ixy="0" ixz="0" iyz="0"/>
-    </inertial>
-  </link>
   <joint name="back_right_shock_joint" type="prismatic">
     <limit lower="0" upper="${shock_travel}" effort="100" velocity="100"/>
@@ -308,48 +355,4 @@
     <limit effort="10000" velocity="500" />
   </joint>
-  <link name="front_left_wheel_shock">
-      <visual>
-      <origin xyz="0 0 0.1" rpy="0 0 0"/>
-      <geometry>
-        <cylinder length="0.2" radius="0.01"/>
-      </geometry>
-      <material name="silver">
-        <color rgba="0.75 0.75 0.75 1"/>
-      </material>
-    </visual>
-    <collision>
-      <origin xyz="0 0 0.1" rpy="0 0 0"/>
-      <geometry>
-        <cylinder length="0.2" radius="0.01"/>
-      </geometry>
-    </collision>
-    <inertial>
-      <mass value="0.01"/>
-      <inertia ixx="0.015" iyy="0.0375" izz="0.0375"
-               ixy="0" ixz="0" iyz="0"/>
-    </inertial>
-  </link>
-    <link name="front_right_wheel_shock">
-      <visual>
-      <origin xyz="0 0 0.1" rpy="0 0 0"/>
-      <geometry>
-        <cylinder length="0.2" radius="0.01"/>
-      </geometry>
-      <material name="silver">
-        <color rgba="0.75 0.75 0.75 1"/>
-      </material>
-    </visual>
-    <collision>
-      <origin xyz="0 0 0.1" rpy="0 0 0"/>
-      <geometry>
-        <cylinder length="0.2" radius="0.01"/>
-      </geometry>
-    </collision>
-    <inertial>
-      <mass value="0.01"/>
-      <inertia ixx="0.015" iyy="0.0375" izz="0.0375"
-               ixy="0" ixz="0" iyz="0"/>
-    </inertial>
-  </link>
   <joint name="front_right_shock_joint" type="prismatic">
     <limit lower="0" upper="${shock_travel}" effort="100" velocity="100"/>

Commit message: Change geometries to make more stable for Nav2

File: car_description/robot/car.urdf.xacro (robot description, xacro)
@@ -115,5 +115,5 @@
     <sensor type="ray" name="laser_scanner">
     <always_on>true</always_on>
-    <visualize>false</visualize>
+    <visualize>true</visualize>
     <update_rate>8</update_rate>
     <ray>
@@ -127,5 +127,5 @@
       </scan>
       <range>
-        <min>0.10</min>
+        <min>0.30</min>
         <max>15.0</max>
         <resolution>0.1</resolution>
@@ -233,5 +233,5 @@
       <origin xyz="0 0 0.1" rpy="0 0 0"/>
       <geometry>
-        <cylinder length="0.2" radius="0.01"/>
+        <cylinder length="0.05" radius="0.01"/>
       </geometry>
       <material name="silver">
@@ -242,5 +242,5 @@
       <origin xyz="0 0 0.1" rpy="0 0 0"/>
       <geometry>
-        <cylinder length="0.2" radius="0.01"/>
+        <cylinder length="0.05" radius="0.01"/>
       </geometry>
     </collision>
@@ -255,5 +255,5 @@
     <origin xyz="0 0 0.1" rpy="0 0 0"/>
     <geometry>
-      <cylinder length="0.2" radius="0.01"/>
+      <cylinder length="0.05" radius="0.01"/>
     </geometry>
     <material name="silver">
@@ -264,5 +264,5 @@
     <origin xyz="0 0 0.1" rpy="0 0 0"/>
     <geometry>
-      <cylinder length="0.2" radius="0.01"/>
+      <cylinder length="0.05" radius="0.01"/>
     </geometry>
   </collision>
@@ -277,5 +277,5 @@
       <origin xyz="0 0 0.1" rpy="0 0 0"/>
       <geometry>
-        <cylinder length="0.2" radius="0.01"/>
+        <cylinder length="0.05" radius="0.01"/>
       </geometry>
       <material name="silver">
@@ -286,5 +286,5 @@
       <origin xyz="0 0 0.1" rpy="0 0 0"/>
       <geometry>
-        <cylinder length="0.2" radius="0.01"/>
+        <cylinder length="0.05" radius="0.01"/>
       </geometry>
     </collision>
@@ -299,5 +299,5 @@
       <origin xyz="0 0 0.1" rpy="0 0 0"/>
       <geometry>
-        <cylinder length="0.2" radius="0.01"/>
+        <cylinder length="0.05" radius="0.01"/>
       </geometry>
       <material name="silver">
@@ -308,5 +308,5 @@
       <origin xyz="0 0 0.1" rpy="0 0 0"/>
       <geometry>
-        <cylinder length="0.2" radius="0.01"/>
+        <cylinder length="0.05" radius="0.01"/>
       </geometry>
     </collision>
